File: pcb/C152Quadrant/C152Quadrant.kicad_pcb (KiCad board)
At the start: 2 copper layers, 140 x 85 mm, 67 parts, among them J1 Conn_02x03_Odd_Even, J2 USB_B_Micro, J3 Conn_02x05_Odd_Even, Q1 BC807, Q2 BC807, SW1 SW_Push, U1 STM32F103C8Tx, U2 MIC5504, U3 74LS125, U4 74LS125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

Commit message: Added PCB gerber files
Routing:
- net GND: track 26.0 -> 35.2 mm, vias 58 -> 59
- net +5V: track 24.8 -> 25.5 mm
Changed lines of the file:
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@@
     (thickness 1.6)
     (drawings 15)
-    (tracks 648)
+    (tracks 653)
     (zones 0)
     (modules 67)
@@
     (visible_elements FFFDFF7F)
     (pcbplotparams
-      (layerselection 0x010fc_ffffffff)
-      (usegerberextensions false)
+      (layerselection 0x010e0_ffffffff)
+      (usegerberextensions true)
       (usegerberattributes true)
       (usegerberadvancedattributes true)
@@
       (outputformat 1)
       (mirror false)
-      (drillshape 1)
+      (drillshape 0)
       (scaleselection 1)
-      (outputdirectory ""))
+      (outputdirectory "gerber/"))
   )
   (net 0 "")
@@
       (effects (font (size 0.8 0.8) (thickness 0.12)))
     )
-    (pad 1 smd roundrect (at -1.5625 0 90) (size 1.325 1.8) (layers F.Cu F.Paste F.Mask) (roundrect_rratio 0.188679)
+    (pad 1 smd roundrect (at -1.5625 0 90) (size 1.325 1.8) (layers F.Cu F.Paste F.Mask) (roundrect_rratio 0.1886784905660377)
       (net 1 GND))
-    (pad 2 smd roundrect (at 1.5625 0 90) (size 1.325 1.8) (layers F.Cu F.Paste F.Mask) (roundrect_rratio 0.188679)
+    (pad 2 smd roundrect (at 1.5625 0 90) (size 1.325 1.8) (layers F.Cu F.Paste F.Mask) (roundrect_rratio 0.1886784905660377)
       (net 12 +5V))
     (model ${KISYS3DMOD}/Capacitor_SMD.3dshapes/C_1206_3216Metric.wrl
@@
       (effects (font (size 0.8 0.8) (thickness 0.12)))
     )
-    (pad 2 smd roundrect (at 1.5625 0 180) (size 1.325 1.8) (layers F.Cu F.Paste F.Mask) (roundrect_rratio 0.188679)
+    (pad 2 smd roundrect (at 1.5625 0 180) (size 1.325 1.8) (layers F.Cu F.Paste F.Mask) (roundrect_rratio 0.1886784905660377)
       (net 13 +3V3))
-    (pad 1 smd roundrect (at -1.5625 0 180) (size 1.325 1.8) (layers F.Cu F.Paste F.Mask) (roundrect_rratio 0.188679)
+    (pad 1 smd roundrect (at -1.5625 0 180) (size 1.325 1.8) (layers F.Cu F.Paste F.Mask) (roundrect_rratio 0.1886784905660377)
       (net 1 GND))
     (model ${KISYS3DMOD}/Capacitor_SMD.3dshapes/C_1206_3216Metric.wrl
@@
   (segment (start 219.65 100.965702) (end 220.359298 101.675) (width 0.25) (layer F.Cu) (net 1))
   (segment (start 219.65 100.1625) (end 219.65 100.965702) (width 0.25) (layer F.Cu) (net 1))
+  (segment (start 232.4 139.2) (end 238 139.2) (width 0.3) (layer F.Cu) (net 1))
+  (segment (start 237.9 139.1) (end 237.9 135.6) (width 0.3) (layer F.Cu) (net 1))
+  (segment (start 238 139.2) (end 237.9 139.1) (width 0.3) (layer F.Cu) (net 1))
+  (via (at 203.2 97.8) (size 0.8) (drill 0.4) (layers F.Cu B.Cu) (net 1))
   (segment (start 120.3625 90.75) (end 120.3625 86) (width 0.25) (layer F.Cu) (net 2))
   (segment (start 106.25 152.5) (end 106.25 107.55) (width 0.4) (layer F.Cu) (net 2))
@@
   (segment (start 207.4 95.8) (end 209.95 93.25) (width 0.25) (layer F.Cu) (net 3))
   (segment (start 146.25 152.5) (end 146.25 108.15) (width 0.4) (layer F.Cu) (net 4))
-  (segment (start 162.0625 92.3375) (end 162.0625 87.4) (width 0.25) (layer F.Cu) (net 4))
+  (segment (start 162.0625 92.3375) (end 162.0625 87.4) (width 0.4) (layer F.Cu) (net 4))
   (segment (start 146.25 108.15) (end 162.0625 92.3375) (width 0.4) (layer F.Cu) (net 4))
-  (segment (start 162.0625 87.4) (end 162.0625 83.2) (width 0.25) (layer F.Cu) (net 4))
-  (segment (start 162.0625 82.1375) (end 162.0625 83.2) (width 0.25) (layer F.Cu) (net 4))
+  (segment (start 162.0625 87.4) (end 162.0625 83.2) (width 0.4) (layer F.Cu) (net 4))
+  (segment (start 162.0625 82.1375) (end 162.0625 83.2) (width 0.4) (layer F.Cu) (net 4))
   (segment (start 164.6 79.6) (end 162.0625 82.1375) (width 0.4) (layer F.Cu) (net 4))
   (segment (start 194.4 79.6) (end 164.6 79.6) (width 0.4) (layer F.Cu) (net 4))
@@
   (segment (start 176.6375 87.25) (end 176.6875 87.2) (width 0.25) (layer F.Cu) (net 11))
   (segment (start 172.38 87.25) (end 176.6375 87.25) (width 0.25) (layer F.Cu) (net 11))
-  (segment (start 176.6875 84.925) (end 178.3625 83.25) (width 0.25) (layer F.Cu) (net 11))
-  (segment (start 176.6875 87.2) (end 176.6875 84.925) (width 0.25) (layer F.Cu) (net 11))
   (segment (start 214.323022 85.65002) (end 205.85002 85.65002) (width 0.25) (layer F.Cu) (net 11))
   (segment (start 217.15 88.476998) (end 214.323022 85.65002) (width 0.25) (layer F.Cu) (net 11))
@@
   (segment (start 178.7125 83.6) (end 178.3625 83.25) (width 0.25) (layer F.Cu) (net 11))
   (segment (start 180.6 83.6) (end 178.7125 83.6) (width 0.25) (layer F.Cu) (net 11))
+  (segment (start 178.3625 84.0375) (end 178.3625 83.25) (width 0.25) (layer F.Cu) (net 11))
+  (segment (start 176.6875 85.7125) (end 178.3625 84.0375) (width 0.25) (layer F.Cu) (net 11))
+  (segment (start 176.6875 87.2) (end 176.6875 85.7125) (width 0.25) (layer F.Cu) (net 11))
   (segment (start 224.35 144.05) (end 226.85 144.05) (width 0.6) (layer F.Cu) (net 12))
   (segment (start 226.85 144.05) (end 226.85 145.95) (width 0.6) (layer F.Cu) (net 12))
-  (segment (start 226.85 144.05) (end 228.95 144.05) (width 0.6) (layer F.Cu) (net 12))
   (segment (start 226.85 145.95) (end 224.35 145.95) (width 0.6) (layer F.Cu) (net 12))
-  (segment (start 228.95 144.05) (end 230.8 142.2) (width 0.6) (layer F.Cu) (net 12))
-  (segment (start 231.4 141.6) (end 230.8 142.2) (width 0.25) (layer F.Cu) (net 12))
+  (segment (start 231.4 141.6) (end 230.8 142.2) (width 0.3) (layer F.Cu) (net 12))
   (segment (start 232.4 141.6) (end 231.4 141.6) (width 0.25) (layer F.Cu) (net 12))
   (via (at 227.6 139) (size 0.8) (drill 0.4) (layers F.Cu B.Cu) (net 12))
@@
   (segment (start 226.85 143.55) (end 226.85 144.05) (width 0.25) (layer F.Cu) (net 12))
   (segment (start 227.2 143.2) (end 226.85 143.55) (width 0.25) (layer F.Cu) (net 12))
+  (segment (start 228.95 144.05) (end 231.3 141.7) (width 0.6) (layer F.Cu) (net 12))
+  (segment (start 226.85 144.05) (end 228.95 144.05) (width 0.6) (layer F.Cu) (net 12))
   (segment (start 220.15 91.8375) (end 220.15 92.75) (width 0.25) (layer F.Cu) (net 13))
   (segment (start 220.65 93.25) (end 221.5625 93.25) (width 0.25) (layer F.Cu) (net 13))
@@
   (segment (start 236.8 93.08) (end 236.8 89.7125) (width 0.25) (layer F.Cu) (net 25))
   (segment (start 223.6375 140.8) (end 222.25 139.4125) (width 0.25) (layer F.Cu) (net 26))
-  (segment (start 232.4 140.8) (end 223.6375 140.8) (width 0.25) (layer F.Cu) (net 26))
-  (segment (start 226.0875 140) (end 232.4 140) (width 0.25) (layer F.Cu) (net 27))
+  (segment (start 232.4 140.8) (end 223.6375 140.8) (width 0.3) (layer F.Cu) (net 26))
+  (segment (start 226.0875 140) (end 232.4 140) (width 0.3) (layer F.Cu) (net 27))
   (segment (start 225.5 139.4125) (end 226.0875 140) (width 0.25) (layer F.Cu) (net 27))
   (segment (start 216 154.14) (end 217.06 155.2) (width 0.25) (layer F.Cu) (net 28))
@@
   (segment (start 225.1875 137.5875) (end 218.65 131.05) (width 0.25) (layer F.Cu) (net 31))
   (segment (start 225.5 137.5875) (end 225.5 135.7125) (width 0.25) (layer F.Cu) (net 31))
-  (segment (start 222.25 135.31875) (end 222.25 137.5875) (width 0.25) (layer F.Cu) (net 32))
-  (segment (start 218.15 131.21875) (end 222.25 135.31875) (width 0.25) (layer F.Cu) (net 32))
-  (segment (start 218.15 100.1625) (end 218.15 131.21875) (width 0.25) (layer F.Cu) (net 32))
+  (segment (start 222.25 135.65) (end 222.25 137.5875) (width 0.25) (layer F.Cu) (net 32))
+  (segment (start 218.15 131.55) (end 222.25 135.65) (width 0.25) (layer F.Cu) (net 32))
+  (segment (start 218.15 100.1625) (end 218.15 131.55) (width 0.25) (layer F.Cu) (net 32))
   (segment (start 219.12501 100.18749) (end 219.15 100.1625) (width 0.25) (layer F.Cu) (net 33))
   (segment (start 219.8 102.4) (end 226.94 102.4) (width 0.25) (layer F.Cu) (net 33))
@@
   (segment (start 204 144.36) (end 212.6475 144.36) (width 0.25) (layer F.Cu) (net 57))
   (via (at 216.6 110.800002) (size 0.8) (drill 0.4) (layers F.Cu B.Cu) (net 57))
-  (segment (start 217.4 111.600002) (end 216.6 110.800002) (width 0.25) (layer F.Cu) (net 57))
-  (segment (start 217.4 137.82949) (end 217.4 111.600002) (width 0.25) (layer F.Cu) (net 57))
-  (segment (start 213.70001 141.52948) (end 217.4 137.82949) (width 0.25) (layer F.Cu) (net 57))
-  (segment (start 213.70001 143.78749) (end 213.70001 141.52948) (width 0.25) (layer F.Cu) (net 57))
-  (segment (start 212.8875 144.6) (end 213.70001 143.78749) (width 0.25) (layer F.Cu) (net 57))
   (segment (start 214.65 97.25) (end 214.67499 97.27499) (width 0.25) (layer F.Cu) (net 57))
   (segment (start 216.6 110.800002) (end 216.6 97.27499) (width 0.25) (layer B.Cu) (net 57))
@@
   (segment (start 214.67499 97.27499) (end 216.6 97.27499) (width 0.25) (layer F.Cu) (net 57))
   (via (at 216.6 97.27499) (size 0.8) (drill 0.4) (layers F.Cu B.Cu) (net 57))
+  (segment (start 217.4 111.600002) (end 216.6 110.800002) (width 0.25) (layer F.Cu) (net 57))
+  (segment (start 217.4 137.6) (end 217.4 111.600002) (width 0.25) (layer F.Cu) (net 57))
+  (segment (start 213.8 141.2) (end 217.4 137.6) (width 0.25) (layer F.Cu) (net 57))
+  (segment (start 213.8 143.6875) (end 213.8 141.2) (width 0.25) (layer F.Cu) (net 57))
+  (segment (start 212.8875 144.6) (end 213.8 143.6875) (width 0.25) (layer F.Cu) (net 57))
   (zone (net 1) (net_name GND) (layer F.Cu) (hatch edge 0.508)
     (connect_pads (clearance 0.508))
